Commit message: Etap 2: costam dziala

File: my_urdf_pkg/urdf/manipulator_model_with_gripper.urdf (robot description, URDF)
Before this commit: robot my_manipulator, 8 links, 7 joints
Joints:
- joint Joint_2: limit lower=-0.785 upper=0.785 effort=1000.0 velocity=0.5 -> lower=-1.4 upper=1.4 effort=1000.0 velocity=0.5
- joint Joint_3: limit lower=-0.785 upper=0.785 effort=1000.0 velocity=0.5 -> lower=-1.4 upper=1.4 effort=1000.0 velocity=0.5
