Commit message: aktualizacja instrukcji, w trakcie projektu 5

File: my_urdf_pkg/urdf/manipulator_model.urdf (robot description, URDF)
Before this commit: robot my_manipulator, 5 links, 4 joints
Links:
- removed link Tool
- added link tool_null
Joints:
- removed joint tool_nul
- added joint tool_null_joint: type fixed, parent Link_3, child tool_null, origin xyz=0 0 0.8 rpy=0 0 0

File: my_urdf_pkg/urdf/manipulator_model_with_gripper.urdf (robot description, URDF)
Before this commit: robot my_manipulator, 8 links, 7 joints
Links:
- removed link Tool
- added link tool_null
Joints:
- removed joint tool_nul
- added joint tool_null_joint: type fixed, parent Link_3, child tool_null, origin xyz=0 0 0.8 rpy=0 0 0
